Commit message: got ros_control to control one actuator

File: src/rolling_robot_description/rolling_robot.urdf (robot description, URDF)
Before this commit: robot rolling_robot, 3 links, 2 joints
Joints:
- joint joint1: limit lower=0.0 upper=2 effort=-1 velocity=-1 -> lower=0.0 upper=2.0 effort=10000000 velocity=1000

Commit message: 6 actuators controllable from ROS

File: src/rolling_robot_description/rolling_robot.urdf (robot description, URDF)
Before this commit: robot rolling_robot, 3 links, 2 joints
Links:
- added link link2, mass 0.1; collision cylinder length=1 radius=0.05; visual cylinder length=1 radius=0.05
- added link link3, mass 0.1; collision cylinder length=1 radius=0.05; visual cylinder length=1 radius=0.05
- added link link4, mass 0.1; collision cylinder length=1 radius=0.05; visual cylinder length=1 radius=0.05
- added link link5, mass 0.1; collision cylinder length=1 radius=0.05; visual cylinder length=1 radius=0.05
- added link link6, mass 0.1; collision cylinder length=1 radius=0.05; visual cylinder length=1 radius=0.05
Joints:
- added joint joint2: type prismatic, parent base_link, child link2, origin xyz=0 0 0, axis 0 0.5 -0.866025, limit lower=0.0 upper=2.0 effort=10000000 velocity=1000
- added joint joint3: type prismatic, parent base_link, child link3, origin xyz=0 0 0, axis 0 1 0, limit lower=0.0 upper=2.0 effort=10000000 velocity=1000
- added joint joint4: type prismatic, parent base_link, child link4, origin xyz=0 0 0, axis 0 0.5 0.866025, limit lower=0.0 upper=2.0 effort=10000000 velocity=1000
- added joint joint5: type prismatic, parent base_link, child link5, origin xyz=0 0 0, axis 0 -0.5 0.866025, limit lower=0.0 upper=2.0 effort=10000000 velocity=1000
- added joint joint6: type prismatic, parent base_link, child link6, origin xyz=0 0 0, axis 0 -1 0, limit lower=0.0 upper=2.0 effort=10000000 velocity=1000

Commit message: added new rhombicuboctahedron geometry with one dimension of actuators

File: src/rolling_robot_description/rolling_robot.urdf (robot description, URDF)
Before this commit: robot rolling_robot, 8 links, 7 joints
Links:
- added link link7, mass 0.1; collision cylinder length=0.1778 radius=0.005; visual cylinder length=0.1778 radius=0.005
- added link link8, mass 0.1; collision cylinder length=0.1778 radius=0.005; visual cylinder length=0.1778 radius=0.005
- link base_link: mass 10 -> 20; geometry collision mesh filename=/home/eric/rolling_robot/rolling_robot_model/rhombicuboctah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 scale=0.025641 0.025641 0.025641; visual mesh filename=/home/eric/rolling_robot/rolling_robot_model/rhombicuboctah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 scale=0.025641 0.025641 0.025641
- link link1: geometry collision cylinder length=0.1778 radius=0.005; visual cylinder length=0.1778 radius=0.005
- link link2: geometry collision cylinder length=0.1778 radius=0.005; visual cylinder length=0.1778 radius=0.005
- link link3: geometry collision cylinder length=0.1778 radius=0.005; visual cylinder length=0.1778 radius=0.005
- link link4: geometry collision cylinder length=0.1778 radius=0.005; visual cylinder length=0.1778 radius=0.005
- link link5: geometry collision cylinder length=0.1778 radius=0.005; visual cylinder length=0.1778 radius=0.005
- link link6: geometry collision cylinder length=0.1778 radius=0.005; visual cylinder length=0.1778 radius=0.005
Joints:
- added joint joint7: type prismatic, parent base_link, child link7, origin xyz=0 0 0, axis 0 -0.923879 0.382683, limit lower=0.0 upper=0.1778 effort=10000000 velocity=1000
- added joint joint8: type prismatic, parent base_link, child link8, origin xyz=0 0 0, axis 0 -0.923879 -0.382683, limit lower=0.0 upper=0.1778 effort=10000000 velocity=1000
- joint joint1: axis 0 -0.5 -0.866025 -> 0 -0.382683 -0.923880; limit lower=0.0 upper=2.0 effort=10000000 velocity=1000 -> lower=0.0 upper=0.1778 effort=10000000 velocity=1000
- joint joint2: axis 0 0.5 -0.866025 -> 0 0.382683 -0.923880; limit lower=0.0 upper=2.0 effort=10000000 velocity=1000 -> lower=0.0 upper=0.1778 effort=10000000 velocity=1000
- joint joint3: axis 0 1 0 -> 0 0.923879 -0.382683; limit lower=0.0 upper=2.0 effort=10000000 velocity=1000 -> lower=0.0 upper=0.1778 effort=10000000 velocity=1000
- joint joint4: axis 0 0.5 0.866025 -> 0 0.923879 0.382683; limit lower=0.0 upper=2.0 effort=10000000 velocity=1000 -> lower=0.0 upper=0.1778 effort=10000000 velocity=1000
- joint joint5: axis 0 -0.5 0.866025 -> 0 0.382683 0.923880; limit lower=0.0 upper=2.0 effort=10000000 velocity=1000 -> lower=0.0 upper=0.1778 effort=10000000 velocity=1000
- joint joint6: axis 0 -1 0 -> 0 -0.382683 0.923880; limit lower=0.0 upper=2.0 effort=10000000 velocity=1000 -> lower=0.0 upper=0.1778 effort=10000000 velocity=1000

Commit message: updated URDF with 16 actuators; added script for open-loop side motion

File: src/rolling_robot_description/rolling_robot.urdf (robot description, URDF)
Before this commit: robot rolling_robot, 10 links, 9 joints
Links:
- added link link10, mass 0.1; collision cylinder length=0.1778 radius=0.005; visual cylinder length=0.1778 radius=0.005
- added link link11, mass 0.1; collision cylinder length=0.1778 radius=0.005; visual cylinder length=0.1778 radius=0.005
- added link link12, mass 0.1; collision cylinder length=0.1778 radius=0.005; visual cylinder length=0.1778 radius=0.005
- added link link13, mass 0.1; collision cylinder length=0.1778 radius=0.005; visual cylinder length=0.1778 radius=0.005
- added link link14, mass 0.1; collision cylinder length=0.1778 radius=0.005; visual cylinder length=0.1778 radius=0.005
- added link link15, mass 0.1; collision cylinder length=0.1778 radius=0.005; visual cylinder length=0.1778 radius=0.005
- added link link16, mass 0.1; collision cylinder length=0.1778 radius=0.005; visual cylinder length=0.1778 radius=0.005
- added link link9, mass 0.1; collision cylinder length=0.1778 radius=0.005; visual cylinder length=0.1778 radius=0.005
Joints:
- added joint joint10: type prismatic, parent base_link, child link10, origin xyz=0 0 0, axis 0.382683 0 -0.923880, limit lower=0.0 upper=0.1778 effort=10000000 velocity=1000
- added joint joint11: type prismatic, parent base_link, child link11, origin xyz=0 0 0, axis 0.923879 0 -0.382683, limit lower=0.0 upper=0.1778 effort=10000000 velocity=1000
- added joint joint12: type prismatic, parent base_link, child link12, origin xyz=0 0 0, axis 0.923879 0 0.382683, limit lower=0.0 upper=0.1778 effort=10000000 velocity=1000
- added joint joint13: type prismatic, parent base_link, child link13, origin xyz=0 0 0, axis 0.382683 0 0.923880, limit lower=0.0 upper=0.1778 effort=10000000 velocity=1000
- added joint joint14: type prismatic, parent base_link, child link14, origin xyz=0 0 0, axis -0.382683 0 0.923880, limit lower=0.0 upper=0.1778 effort=10000000 velocity=1000
- added joint joint15: type prismatic, parent base_link, child link15, origin xyz=0 0 0, axis -0.923879 0 0.382683, limit lower=0.0 upper=0.1778 effort=10000000 velocity=1000
- added joint joint16: type prismatic, parent base_link, child link16, origin xyz=0 0 0, axis -0.923879 0 -0.382683, limit lower=0.0 upper=0.1778 effort=10000000 velocity=1000
- added joint joint9: type prismatic, parent base_link, child link9, origin xyz=0 0 0, axis -0.382683 0 -0.923880, limit lower=0.0 upper=0.1778 effort=10000000 velocity=1000

Commit message: added imu and started state estimation package

File: src/rolling_robot_description/rolling_robot.urdf (robot description, URDF)
Before this commit: robot rolling_robot, 18 links, 17 joints
Links:
- added link imu_link, mass 0.001; collision box size=.001 .001 .001; visual box size=0.001 0.001 0.001
Joints:
- added joint imu_joint: type fixed, parent base_link, child imu_link

Commit message: added uwb_interface package to get positions of simulated uwb links

File: src/rolling_robot_description/rolling_robot.urdf (robot description, URDF)
Before this commit: robot rolling_robot, 19 links, 18 joints
Links:
- added link uwb_link1, mass 0.00001; collision box size=.01 .01 .01; visual box size=0.01 0.01 0.01
- added link uwb_link2, mass 0.00001; collision box size=0.01 0.01 0.01; visual box size=0.01 0.01 0.01
- link imu_link: geometry collision box size=.01 .01 .01; visual box size=0.01 0.01 0.01
Joints:
- added joint uwb_joint1: type revolute, parent base_link, child uwb_link1, origin xyz=0.2 0 0 rpy=0 0 0, axis 0 0 0, limit lower=0 upper=0 effort=0 velocity=0
- added joint uwb_joint2: type revolute, parent base_link, child uwb_link2, origin xyz=-0.2 0 0 rpy=0 0 0, axis 0 0 0, limit lower=0 upper=0 effort=0 velocity=0
- joint imu_joint: axis (none) -> 0 0 0; limit (none) -> lower=0 upper=0 effort=0 velocity=0; origin (none) -> xyz=0 0 0 rpy=0 0 0; type fixed -> revolute

Commit message: added .gitignore, added orientation estimation using 3 UWB measurements

File: src/rolling_robot_description/rolling_robot.urdf (robot description, URDF)
Before this commit: robot rolling_robot, 21 links, 20 joints
Links:
- added link uwb_link3, mass 0.00001; collision box size=0.01 0.01 0.01; visual box size=0.01 0.01 0.01
Joints:
- added joint uwb_joint3: type revolute, parent base_link, child uwb_link3, origin xyz=-0.21 0.21 0 rpy=0 0 0, axis 0 0 0, limit lower=0 upper=0 effort=0 velocity=0
- joint uwb_joint1: origin xyz=0.2 0 0 rpy=0 0 0 -> xyz=-0.21 -0.21 0 rpy=0 0 0
- joint uwb_joint2: origin xyz=-0.2 0 0 rpy=0 0 0 -> xyz=0.21 -0.21 0 rpy=0 0 0
